File: PCB/BigFoot.kicad_sch (KiCad schematic)
At the start: 28 parts

Commit message: Final PCB Version
Parts:
- removed D1, D2, D3, D4, D5, D6, D7, D8: LED, symbol Device:LED
- added ExprPedalJack1, ExprPedalJack2: ACJS-IH, Connectors:Jack_6.35_Horizontal_Amphenol_ACJS-IH, symbol Connector:AudioJack3
- added LedSW0, LedSW1, LedSW2, LedSW3, LedSW4, LedSW5, LedSW6, LedSW7, StateLED1: TLHR4400-AS12Z, LED_THT:LED_D3.0mm, symbol Device:LED
- added R10, R11, R3, R4, R5, R6, R7, R8, R9: 47, Resistor_THT:R_Axial_DIN0309_L9.0mm_D3.2mm_P15.24mm_Horizontal, symbol Device:R
- added TRS/RTS_Switch1, TRS/RTS_Switch2: LSSA22L-V, Switch:Switch_slide_2PDT_LSSA22L-V, symbol Switch:SW_Push_DPDT
- MidiOut1: renamed from J?; value Midi Out -> KCDX-5S-S2; footprint (none) -> Connectors:Circular_DIN_5P_KCDX-5S-S2
- R1, R2: renamed from R?; footprint (none) -> Resistor_THT:R_Axial_DIN0309_L9.0mm_D3.2mm_P15.24mm_Horizontal
- U1, U2: renamed from U?; value 74HC4051 -> CD74HCT4051E; footprint (none) -> Package_DIP:DIP-16_W7.62mm
- gave numbers to parts that had none: 15
Connections:
- net +3.3V: now also TRS/RTS_Switch1.5 (B), TRS/RTS_Switch2.5 (B)
- net GND: now also ExprPedalJack1.S, ExprPedalJack2.S, LedSW0.1 (K), LedSW1.1 (K), LedSW2.1 (K), LedSW3.1 (K), LedSW4.1 (K), LedSW5.1 (K), LedSW6.1 (K), LedSW7.1 (K), StateLED1.1 (K); no longer U3.17 (GND)
- net at U2.1 (A4): now also R5.2
- net at U2.12 (A3): now also R8.2
- net at U2.13 (A0): now also R3.2
- net at U2.14 (A1): now also R7.2
- net at U2.15 (A2): now also R4.2
- net at U2.2 (A6): now also R6.2
- net at U2.4 (A7): now also R10.2
- net at U2.5 (A5): now also R9.2
- net at U3.20 (13_LED_SCK0): now also R11.2
- net ExprPedal1: now reaches U3.21 (14_A0_SCK0)
- net ExprPedal1: now also TRS/RTS_Switch1.2 (B)
- net ExprPedal2: now reaches U3.22 (15_A1_Touch)
- net ExprPedal2: now also TRS/RTS_Switch2.2 (B)
- new net: LedSW0.2 (A), R3.1
- new net: ExprPedalJack1.T, TRS/RTS_Switch1.1 (A), TRS/RTS_Switch1.6 (C)
- new net: ExprPedalJack1.R, TRS/RTS_Switch1.3 (C), TRS/RTS_Switch1.4 (A)
- new net: ExprPedalJack2.T, TRS/RTS_Switch2.1 (A), TRS/RTS_Switch2.6 (C)
- new net: ExprPedalJack2.R, TRS/RTS_Switch2.3 (C), TRS/RTS_Switch2.4 (A)
- new net: LedSW3.2 (A), R8.1
- new net: LedSW2.2 (A), R4.1
- new net: LedSW7.2 (A), R10.1
- new net: LedSW1.2 (A), R7.1
- new net: LedSW5.2 (A), R9.1
- new net: LedSW4.2 (A), R5.1
- new net: R11.1, StateLED1.2 (A)
- new net: LedSW6.2 (A), R6.1
- no-connect marks 12 -> 37
Other:
- note added: "- TODO: Display - TODO: Alimentation - TODO: I²C connector"
- note added: "Expression Pedals"
- note added: "Foot Switches - TODO: LEDS"
- note removed: "- TODO: Expression Pedal Input - TODO: Display"
- note removed: "Foot Switches - Finish ordering - TODO: LEDS"
- title: (none) -> BigFoot
- moved on the sheet: BankSwitch+1, BankSwith-1, MidiOut1, R1, R2, U3
