File: PCB/BigFoot.kicad_pcb (KiCad board)
At the start: 2 copper layers, 235 x 96.5 mm, 42 parts, among them U1 74HCT4051, U2 74HCT4051, U3 Teensy-LC

Commit message: Pre Release version
Parts:
- added G***: LOGO, LOGO, F.Cu at (239.2, 124.1)

Commit message: Version 3.0
Other:
- board text added: "https://github.com/pierre-girbon/BigFoot CC BY-NC 4.0"
Changed lines of the file:
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@@
       (viasonmask false)
       (mode 1)
-      (useauxorigin false)
+      (useauxorigin true)
       (hpglpennumber 1)
       (hpglpenspeed 20)
@@
     (effects (font (size 2 2) (thickness 0.3)))
   )
+  (gr_text "https://github.com/pierre-girbon/BigFoot\nCC BY-NC 4.0" (at 54.22 99) (layer "F.SilkS")
+    (effects (font (size 1 1) (thickness 0.15)) (justify left))
+  )
   (gr_text "Rev3" (at 57.36 91.76) (layer "F.SilkS")
