File: Enclosure/BigFoot-Enclosure/BigFoot-Enclosure.kicad_pcb (KiCad board)
At the start: 2 copper layers, 247 x 108.5 mm, 27 parts, among them Sw1 MountingHole, Sw2 MountingHole, Sw3 MountingHole, Sw4 MountingHole, Sw5 MountingHole, Sw6 MountingHole, Sw7 MountingHole, Sw8 MountingHole

Commit message: Pre Release version
Changed lines of the file:
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@@
   (gr_line locked (start 274.2 150.5) (end 27.2 150.5) (layer "Edge.Cuts") (width 0.1))
   (gr_line locked (start 94.7 48) (end 94.7 42) (layer "Edge.Cuts") (width 0.1))
-  (gr_text "Expr2" (at 246.3 45.5) (layer "F.SilkS")
+  (gr_text "Expr1" (at 246.3 45.5) (layer "F.SilkS")
     (effects (font (size 1.5 1.5) (thickness 0.375)))
   )
@@
     (effects (font (size 2 2) (thickness 0.3)))
   )
-  (gr_text "Expr1" (at 198.1 45.5) (layer "F.SilkS")
+  (gr_text "Expr2" (at 198.1 45.5) (layer "F.SilkS")
     (effects (font (size 1.5 1.5) (thickness 0.375)))
   )
